File: hardware/PCB/rev01/rev01.kicad_sch (KiCad schematic)
At the start: 63 parts, among them J3 Conn_Coaxial, J4 USB_C_Receptacle_USB2.0_16P, J5 GPS_ANT, Q4 DMG3415U, SW1 RESET, SW2 BOOT, U1 NEO-M8N, U2 ESP32-S3-WROOM-1, U3 SGTL5000XNLA3, U4 MAX17048G+T10, U5 SA818S, U6 MCP73831T-2ACI/OT, U7 AP2112K-3.3

Commit message: PCB rev01 progress
Parts:
- removed BT1: BR-1225A/FAN, Battery:BatteryHolder_Keystone_3000_1x12mm, symbol Device:Battery_Cell
- removed BT2: 18650_LiIon, Battery:BatteryHolder_Keystone_1042_1x18650, symbol Device:Battery_Cell
- removed C1, C3, C5: 10u, Capacitor_SMD:C_0603_1608Metric, symbol Device:C
- removed C10: 100u_SA818, Capacitor_SMD:C_1206_3216Metric, symbol Device:C
- removed C11: 100n_VDDD, Capacitor_SMD:C_0402_1005Metric, symbol Device:C
- removed C12: 100n_VDDA, Capacitor_SMD:C_0402_1005Metric, symbol Device:C
- removed C13: 100n_VDDIO, Capacitor_SMD:C_0402_1005Metric, symbol Device:C
- removed C14: 1u_VAG, Capacitor_SMD:C_0603_1608Metric, symbol Device:C
- removed C15: 100n_CPFLT, Capacitor_SMD:C_0402_1005Metric, symbol Device:C
- removed C16: 1u_AF_RX_IN, Capacitor_SMD:C_0603_1608Metric, symbol Device:C
- removed C17: 1u_AF_TX_OUT, Capacitor_SMD:C_0603_1608Metric, symbol Device:C
- removed C18: 100n_FG_VDD, Capacitor_SMD:C_0402_1005Metric, symbol Device:C
- removed C19: 4.7u_CHG_IN, Capacitor_SMD:C_0603_1608Metric, symbol Device:C
- removed C2, C25, C4, C6: 100n, Capacitor_SMD:C_0402_1005Metric, symbol Device:C
- removed C20: 4.7u_CHG_BAT, Capacitor_SMD:C_0603_1608Metric, symbol Device:C
- removed C21: 100n_EN_DELAY, Capacitor_SMD:C_0402_1005Metric, symbol Device:C
- removed C22: 10u_3V3_ENTRY, Capacitor_SMD:C_0603_1608Metric, symbol Device:C
- removed C23: 10u_VHI_IN, Capacitor_SMD:C_0603_1608Metric, symbol Device:C
- removed C24: 10u_3V3_OUT, Capacitor_SMD:C_0603_1608Metric, symbol Device:C
- removed C7: 4.7u_GPS_BULK, Capacitor_SMD:C_0603_1608Metric, symbol Device:C
- removed C8: 100n_SA818, Capacitor_SMD:C_0402_1005Metric, symbol Device:C
- removed C9: 10u_SA818, Capacitor_SMD:C_0603_1608Metric, symbol Device:C
- removed D1: LED_CHG, LED_SMD:LED_0603_1608Metric, symbol Device:LED
- removed D2: BAT54, Diode_SMD:D_SOD-323, symbol Device:D
- removed D5: TVS_USB_IN, Diode_SMD:D_SOD-323, symbol Device:D
- removed D6: MBR0540, Diode_SMD:D_SOD-123, symbol Device:D
- removed FB2: FB_SGTL_VDDA, Inductor_SMD:L_0603_1608Metric, symbol Device:R
- removed J3: Conn_Coaxial, Connector_Coaxial:SMA_Amphenol_132134-11_Vertical, symbol Connector:Conn_Coaxial
- removed J4: USB_C_Receptacle_USB2.0_16P, Connector_USB:USB_C_Receptacle_GCT_USB4105-xx-A_16P_TopMnt_Horizontal, symbol Connector:USB_C_Receptacle_USB2.0_16P
- removed J5: GPS_ANT, Connector_Coaxial:U.FL_Hirose_U.FL-R-SMT-1_Vertical, symbol Connector:Conn_Coaxial
- removed Q4: DMG3415U, Package_TO_SOT_SMD:SOT-23, symbol Device:Q_PMOS
- removed R1, R2: 10k, Resistor_SMD:R_0402_1005Metric, symbol Device:R
- removed R10: 10k_ALRT_PU, Resistor_SMD:R_0402_1005Metric, symbol Device:R
- removed R11: 0R_QSTRT_GND, Resistor_SMD:R_0402_1005Metric, symbol Device:R
- removed R12: 10k_STAT_PU, Resistor_SMD:R_0402_1005Metric, symbol Device:R
- removed R13: 10k_EN_PULLUP, Resistor_SMD:R_0402_1005Metric, symbol Device:R
- removed R14: 10k_IO0_PULLUP, Resistor_SMD:R_0402_1005Metric, symbol Device:R
- removed R15: 5.1k_CC1, Resistor_SMD:R_0402_1005Metric, symbol Device:R
- removed R16: 5.1k_CC2, Resistor_SMD:R_0402_1005Metric, symbol Device:R
- removed R17: 4.7k_GPS_BCKP_CHG, Resistor_SMD:R_0402_1005Metric, symbol Device:R
- removed R19: 100k_VBUS_PD, Resistor_SMD:R_0402_1005Metric, symbol Device:R
- removed R21: 100k_EN_PULLUP, Resistor_SMD:R_0402_1005Metric, symbol Device:R
- removed R3, R4: 4.7k, Resistor_SMD:R_0402_1005Metric, symbol Device:R
- removed R5: 1k_RPROG, Resistor_SMD:R_0603_1608Metric, symbol Device:R
- removed R7: 47k_PTT_PULLUP, Resistor_SMD:R_0402_1005Metric, symbol Device:R
- removed R8: 10k_PD_PULLUP, Resistor_SMD:R_0402_1005Metric, symbol Device:R
- removed R9: DNP, Resistor_SMD:R_0402_1005Metric, symbol Device:R
- removed SW1: RESET, Button_Switch_SMD:SW_SPST_TL3342, symbol Switch:SW_Push
- removed SW2: BOOT, Button_Switch_SMD:SW_SPST_TL3342, symbol Switch:SW_Push
- removed U1: NEO-M8N, PAKT_GPS_Fp:ublox_NEO, symbol PAKT_GPS_Sym:NEO-M8N
- removed U2: ESP32-S3-WROOM-1, PAKT_RF_Module_Fp:ESP32-S3-WROOM-1, symbol PAKT_RF_Module_Sym:ESP32-S3-WROOM-1
- removed U3: SGTL5000XNLA3, PAKT_Audio_Fp:QFN-32-1EP_5x5mm_P0.5mm_EP3.6x3.6mm, symbol PAKT_Audio_Sym:SGTL5000XNLA3
- removed U4: MAX17048G+T10, PAKT_MAX17048_Fp:DFN-8-1EP_3x2mm_P0.5mm_EP1.7x1.4mm, symbol PAKT_MAX17048_Sym:MAX17048
- removed U5: SA818S, PAKT_SA818_Fp:XCVR_SA818S, symbol PAKT_SA818_Sym:SA818S
- removed U6: MCP73831T-2ACI/OT, Package_TO_SOT_SMD:SOT-23-5, symbol PAKT_MCP73831_Sym:MCP73831T-2ACI/OT
- removed U7: AP2112K-3.3, Package_TO_SOT_SMD:SOT-23-5, symbol Regulator_Linear:AP2204K-1.5
Connections:
- no-connect marks 12 -> 0
Other:
- added sheet ESP_USB_POWER (rev01_esp_usb_power.kicad_sch)
- added sheet GPS (rev01_gps.kicad_sch)
- added sheet SGTL_SA818 (rev01_sgtl_sa818.kicad_sch)
- title: (none) -> PAKT rev01 - Top

Commit message: pcb progress
Parts:
- added H1, H2, H3, H4: MountingHole_Pad, MountingHole:MountingHole_3.2mm_M3_Pad, symbol Mechanical:MountingHole_Pad
Connections:
- new net GND: H1.1, H2.1, H3.1, H4.1
