File: hardware/PCB/rev01/rev01_sgtl_sa818.kicad_sch (KiCad schematic)
At the start: 24 parts, among them J2 CONSMA006.062, U3 SGTL5000XNLA3, U5 SA818S, U9 0500LP15A500E

Commit message: pcb progress
Parts:
- added U10: AP7313-15SAG-7, PAKT_AP7313_Fp:AP7313_15SAG_7, symbol PAKT_AP7313_Sym:AP7313-15SAG-7
- C11, C12, C13, C15, C8: footprint Capacitor_SMD:C_0402_1005Metric -> Capacitor_SMD:C_0603_1608Metric
- C33: footprint HAm_Extension_Footprints:CAP_EEEFK1A151P -> PAKT_Local_Fp:CAP_EEEFK1A151P
- C9: footprint Capacitor_SMD:C_0603_1608Metric -> Capacitor_SMD:C_0805_2012Metric
- J2: footprint HAm_Extension_Footprints:TE_CONSMA006.062 -> PAKT_Local_Fp:SMA_Amphenol_132134-14_Vertical_P5
- R7, R8, R9: footprint Resistor_SMD:R_0402_1005Metric -> Resistor_SMD:R_0603_1608Metric
- U3: footprint PAKT_Audio_Fp:QFN-32-1EP_5x5mm_P0.5mm_EP3.6x3.6mm -> PAKT_Audio_Fp:HUQFN20_SOT1628-1_NXP
- U9: footprint HAm_Extension_Footprints:0500LP15A500E_JOT -> PAKT_Local_Fp:0500LP15A500E_JOT; symbol 0500LP15A500E_JOT:0500LP15A500E -> Filter_1411-5_1.4x1.1mm:0500LP15A500E
Connections:
- net +3.3V: now also U10.1 (IN); no longer C11.1, C12.1, C6.1, FB2.1, U3.20 (VDDD), U3.3 (VDDA)
- net +5V_SA818: no longer C33.1
- net GND: now also C15.1, U10.3 (GND); no longer C15.2
- net at C10.1, C8.1, C9.1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: now also C33.1
- net at U3.5 (VAG): now also C15.2; no longer C15.1
- new net: C11.1, U10.2 (OUT), U3.20 (VDDD)
- new net VDDA: C12.1, C6.1, FB2.1, U3.3 (VDDA)
Other:
- moved on the sheet: C15, C33, D15, R9

Commit message: progress on pcb
Parts:
- R9: now not fitted
Other:
- moved on the sheet: C11, C15, C16, C17, C4, C5, J2, U10, U3, U9
